File: Circuitos/Circuito de Motores y Alimentación/CircuitoMA_Tesis/Prototipo_2X_DobleCapa.brd (EAGLE design)
At the start: 74 x 84 mm, 33 parts, among them Q1 IRLZ44Z, Q2 IRLZ44Z, Q3 IRLZ44Z, Q4 IRLZ44Z, X1 22-23-2021

Commit message: Circuito
Parts:
- removed POWER, VCC: SPST, gm-switches:SPST
- removed X1: 22-23-2021, con-molex:22-23-2021
- added JP1: (no value), pinhead:1X02
- added JP2: (no value), pinhead:1X02/90
- moved MOTORES 2.69 mm to (51.1, 6.78)
- moved H4 2.24 mm to (69.0, 80.0)
- moved H2 2.06 mm to (6.50, 80.0)
- moved C4 1.58 mm to (16.5, 75.5)
- moved Q4 1.12 mm to (16.4, 31.6)
- moved +11,1V__BATERIA 1.12 mm to (28.7, 9.54)
- moved ARDUINO 1.12 mm to (54.0, 74.5)
- moved C1 1.12 mm to (22.0, 72.5)
- moved C2 1.12 mm to (22.0, 75.5)
- moved C3 1.12 mm to (22.0, 69.5)
- moved D1 1.12 mm to (58.9, 27.6)
- moved D2 1.12 mm to (40.9, 27.3)
- moved D3 1.12 mm to (8.35, 28.0)
- moved D4 1.12 mm to (24.5, 27.6)
- moved GND__BATERIA 1.12 mm to (18.0, 9.54)
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Connections:
- removed net N$6: C4.1, LM7809.OUT, POWER.2
- net GND: now also JP2.1; no longer X1.1
- net N$18: now also C4.1, JP2.2, LM7809.OUT; no longer POWER.1, X1.2
- net N$20: now also JP1.1; no longer VCC.2
- net N$7: now also JP1.2; no longer VCC.1
Routing:
- net N$6: track 35.3 -> 0.00 mm
- net N$18: track 6.13 -> 34.6 mm
- net GND: track 258.8 -> 263.6 mm
- net N$12: track 203.3 -> 207.2 mm
- net N$14: track 62.6 -> 65.6 mm
- net N$15: track 98.4 -> 101.2 mm
- net N$17: track 61.9 -> 64.4 mm
- net N$7: track 9.07 -> 11.4 mm
- net N$20: track 13.4 -> 15.0 mm
Other:
- board size 74 x 84 mm -> 75.5 x 86.5 mm

Commit message: Circuito
Parts:
- added R5, R6, R7, R8: 470KOhm, resistor:0207/7
- R1, R2, R3, R4: value 10kOhm -> 10Ohm
- moved R2 1.12 mm to (54.0, 45.0)
- moved R3 1.12 mm to (32.5, 45.0)
- moved R4 1.00 mm to (24.0, 44.5)
- moved R1 0.50 mm to (65.0, 45.0)
Connections:
- new net N$19: OK2.6, R5.2
- new net N$21: OK3.6, R6.2
- new net N$22: OK4.6, R8.2
- new net N$6: OK1.6, R7.2
- net GND: now also R5.1, R6.1, R7.1, R8.1
Routing:
- net GND: track 263.6 -> 298.2 mm
- net N$19: track 0.00 -> 3.51 mm
- net N$11: track 26.2 -> 22.7 mm
- net N$21: track 0.00 -> 3.46 mm
- net N$22: track 0.00 -> 3.44 mm
- net N$6: track 0.00 -> 3.44 mm
- net N$10: track 30.8 -> 29.0 mm
- net N$9: track 20.8 -> 20.0 mm
- net N$8: track 22.2 -> 22.7 mm

Commit message: Circuito
Parts:
- R1, R2, R3, R4: value 10Ohm -> 1KOhm
- moved D3 16.0 mm to (24.4, 28.0)
- moved D4 16.0 mm to (8.46, 27.6)
Routing:
- net N$16: track 76.8 -> 105.3 mm
- net N$15: track 101.2 -> 81.5 mm
- net N$12: track 207.2 -> 200.5 mm
- net GND: track 298.2 -> 293.1 mm
- net N$8: track 22.7 -> 21.6 mm
