File: Circuitos/Circuito de Motores y Alimentación/CircuitoMA_Tesis/Prototipo_2X_DobleCapa.brd (EAGLE design)
At the start: 75.5 x 86.5 mm, 36 parts, among them Q1 IRLZ44Z, Q2 IRLZ44Z, Q3 IRLZ44Z, Q4 IRLZ44Z

Commit message: Circuito
Routing:
- net N$15: track 81.5 -> 88.3 mm
- net GND: track 293.1 -> 293.7 mm
Changed lines of the file:
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@@
 <layer number="17" name="Pads" color="2" fill="1" visible="yes" active="yes"/>
 <layer number="18" name="Vias" color="2" fill="1" visible="yes" active="yes"/>
-<layer number="19" name="Unrouted" color="6" fill="1" visible="no" active="yes"/>
+<layer number="19" name="Unrouted" color="6" fill="1" visible="yes" active="yes"/>
 <layer number="20" name="Dimension" color="15" fill="1" visible="yes" active="yes"/>
 <layer number="21" name="tPlace" color="7" fill="1" visible="yes" active="yes"/>
@@
 <wire x1="50" y1="59" x2="61" y2="59" width="1.9304" layer="16"/>
 <wire x1="61" y1="59" x2="61.25" y2="58.75" width="0.8128" layer="16"/>
-<wire x1="65" y1="41.19" x2="65" y2="38.18" width="1.9304" layer="16"/>
-<wire x1="65" y1="38.18" x2="64.78" y2="37.96" width="1.6764" layer="16"/>
+<wire x1="65" y1="41.19" x2="64.5" y2="37.68" width="1.9304" layer="16"/>
+<wire x1="64.5" y1="37.68" x2="64.78" y2="37.96" width="1.6764" layer="16"/>
 <contactref element="JP2" pad="1"/>
 <wire x1="13.88" y1="37.96" x2="13.96" y2="37.96" width="1.6764" layer="16"/>
@@
 <wire x1="54.94" y1="54.94" x2="54.94" y2="51.56" width="0.8128" layer="16"/>
 <wire x1="54.94" y1="51.56" x2="56" y2="49.5" width="0.8128" layer="16"/>
-<wire x1="56" y1="49.5" x2="56" y2="47" width="0.8128" layer="16"/>
-<wire x1="56" y1="47" x2="55" y2="46.5" width="0.8128" layer="16"/>
-<wire x1="55" y1="46.5" x2="51" y2="46.5" width="0.8128" layer="16"/>
-<wire x1="51" y1="46.5" x2="49" y2="44.5" width="0.8128" layer="16"/>
-<wire x1="49.02" y1="37.96" x2="49.02" y2="44.48" width="0.8128" layer="16"/>
-<wire x1="49.02" y1="44.48" x2="49" y2="44.5" width="0.8128" layer="16"/>
+<wire x1="56" y1="49.5" x2="56" y2="46" width="0.8128" layer="16"/>
+<wire x1="56" y1="46" x2="55" y2="45" width="0.8128" layer="16"/>
+<wire x1="55" y1="45" x2="51" y2="45" width="0.8128" layer="16"/>
+<wire x1="51" y1="45" x2="49" y2="43" width="0.8128" layer="16"/>
+<wire x1="49.02" y1="37.96" x2="49.02" y2="41.48" width="0.8128" layer="16"/>
+<wire x1="49.02" y1="41.48" x2="49" y2="43" width="0.8128" layer="16"/>
 </signal>
 <signal name="N$15">
@@
 <contactref element="MOTORES" pad="6"/>
 <contactref element="OK3" pad="5"/>
-<wire x1="32.72" y1="37.96" x2="32.72" y2="36.28" width="0.8128" layer="1"/>
-<wire x1="32.72" y1="36.28" x2="34.5" y2="33.5" width="0.8128" layer="1"/>
-<wire x1="34.5" y1="33.5" x2="37.5" y2="33.5" width="0.8128" layer="1"/>
-<wire x1="37.5" y1="33.5" x2="38" y2="34.5" width="0.8128" layer="1"/>
-<wire x1="38" y1="34.5" x2="38" y2="38" width="0.8128" layer="1"/>
+<wire x1="34" y1="30" x2="36.5" y2="30" width="0.8128" layer="1"/>
+<wire x1="36.5" y1="30" x2="38" y2="32" width="0.8128" layer="1"/>
+<wire x1="38" y1="32" x2="38" y2="38" width="0.8128" layer="1"/>
 <wire x1="38" y1="38" x2="43" y2="43" width="0.8128" layer="1"/>
 <wire x1="43" y1="43" x2="43" y2="54.84" width="0.8128" layer="1"/>
@@
 <wire x1="36" y1="24.5" x2="32.5" y2="28" width="1.9304" layer="16"/>
 <wire x1="32.5" y1="28" x2="32.5" y2="32" width="1.9304" layer="16"/>
+<wire x1="32.72" y1="37.96" x2="32.72" y2="31.78" width="0.8128" layer="1"/>
+<wire x1="32.72" y1="31.78" x2="34" y2="30" width="0.8128" layer="1"/>
 </signal>
 <signal name="N$16">
