File: Circuitos/Circuito de Motores y Alimentación/CircuitoMA_Tesis/Prototipo_3X.sch (EAGLE design)
At the start: 18 parts, among them Q1 IRLZ44Z, Q2 IRLZ44Z, Q3 IRLZ44Z, Q4 IRLZ44Z

Commit message: Circuitos y documento
Circuito de control de motores.
Parts:
- removed D5, D6, D7, D8: 1N5817, gm-diodes:1N5817
- added OK1, OK2, OK3, OK4: 4N35, optocoupler:4N35
- added R1, R2, R3, R4: 390 Ohm, resistor:R-US_0207/7
- added R5, R6, R7, R8: 510 Ohm, resistor:R-US_0207/7
Connections:
- new net N$13: Q3.G, R3.1, R7.1
- new net N$17: Q2.G, R2.1, R6.1
- new net N$18: OK1.C, OK2.C, OK3.C, OK4.C
- new net N$5: OK1.EMI, R1.2
- new net N$7: OK2.EMI, R2.2
- net GND: now also R5.2, R6.2, R7.2, R8.2
- net N$1: now also OK1.A; no longer D5.A
- net N$10: now also R4.1, R8.1; no longer D8.C
- net N$11: now also OK1.COL, OK2.COL, OK3.COL, OK4.COL
- net N$2: now also OK2.A; no longer D6.A
- net N$3: now also OK3.A; no longer D7.A
- net N$4: now also OK4.A; no longer D8.A
- net N$6: now also R1.1, R5.1; no longer D5.C
- net N$8: now also OK3.EMI, R3.2; no longer D6.C, Q2.G
- net N$9: now also OK4.EMI, R4.2; no longer D7.C, Q3.G
