File: Circuitos/Circuito de Motores y Alimentación/CircuitoMA_Tesis/Prototipo_3X.brd (EAGLE design)
At the start: 75.5 x 86.5 mm, 18 parts, among them Q1 IRLZ44Z, Q2 IRLZ44Z, Q3 IRLZ44Z, Q4 IRLZ44Z

Commit message: Circuitos y documento
Circuito de control de motores.
Parts:
- removed D5, D6, D7, D8: 1N5817, gm-diodes:DO41-3
- added OK1, OK2, OK3, OK4: 4N35, optocoupler:DIL06
- added R1, R2, R3, R4: 390 Ohm, resistor:0207/7
- added R5, R6, R7, R8: 510 Ohm, resistor:0207/7
- moved D3 43.0 mm to (17.5, 68.0), turned to 90 degrees
- moved Q4 33.6 mm to (10.9, 29.6), turned to 180 degrees
- moved Q2 23.3 mm to (48.0, 30.1), turned to 180 degrees
- moved D1 22.0 mm to (17.5, 53.0), turned to 90 degrees
- moved Q3 20.6 mm to (30.2, 28.6), turned to 180 degrees
- moved Q1 9.91 mm to (64.3, 30.1), turned to 180 degrees
Connections:
- new net N$13: Q3.G, R3.1, R7.1
- new net N$17: Q2.G, R2.1, R6.1
- new net N$18: OK1.2, OK2.2, OK3.2, OK4.2
- new net N$5: OK1.4, R1.2
- new net N$7: OK2.4, R2.2
- net GND: now also R5.2, R6.2, R7.2, R8.2
- net N$1: now also OK1.1; no longer D5.A
- net N$10: now also R4.1, R8.1; no longer D8.C
- net N$11: now also OK1.5, OK2.5, OK3.5, OK4.5
- net N$2: now also OK2.1; no longer D6.A
- net N$3: now also OK3.1; no longer D7.A
- net N$4: now also OK4.1; no longer D8.A
- net N$6: now also R1.1, R5.1; no longer D5.C
- net N$8: now also OK3.4, R3.2; no longer D6.C, Q2.G
- net N$9: now also OK4.4, R4.2; no longer D7.C, Q3.G

Commit message: Circuito Impreso
Parts:
- moved D3 65.3 mm to (59.5, 18.0), turned to 270 degrees
- moved R8 42.6 mm to (22.5, 53.5)
- moved R5 40.5 mm to (53.0, 51.0), turned to 270 degrees
- moved D1 38.9 mm to (28.0, 15.5), turned to 180 degrees
- moved R3 33.1 mm to (10.0, 58.5), turned to 0 degrees
- moved R7 24.0 mm to (10.0, 54.5), turned to 0 degrees
- moved +11,1V__BATERIA 21.2 mm to (8.16, 15.0), turned to 180 degrees
- moved GND__BATERIA 16.8 mm to (8.04, 23.0)
- moved Q3 14.4 mm to (25.2, 42.1)
- moved Q4 13.0 mm to (10.4, 42.6)
- moved Q1 12.5 mm to (63.3, 42.6)
- moved R2 12.3 mm to (43.5, 58.5), turned to 0 degrees
- moved R6 11.4 mm to (43.5, 53.0), turned to 0 degrees
- moved R4 10.8 mm to (22.5, 57.5), turned to 0 degrees
- moved R1 10.0 mm to (57.0, 58.0), turned to 0 degrees
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Connections:
- removed net N$18: OK1.2, OK2.2, OK3.2, OK4.2
- net GND: now also OK1.2, OK2.2, OK3.2, OK4.2
Routing:
- net GND: track 0.00 -> 247.5 mm
- net N$11: track 0.00 -> 155.0 mm
- net N$12: track 0.00 -> 102.4 mm
- net N$16: track 0.00 -> 100.9 mm
- net N$17: track 0.00 -> 66.8 mm
- net N$15: track 0.00 -> 60.6 mm
- net N$14: track 0.00 -> 51.5 mm
- net N$13: track 0.00 -> 39.1 mm
- net N$8: track 0.00 -> 36.8 mm
- net N$6: track 0.00 -> 21.3 mm
- net N$4: track 0.00 -> 16.0 mm
- net N$1: track 0.00 -> 14.6 mm
- net N$10: track 0.00 -> 13.8 mm
- net N$9: track 0.00 -> 12.7 mm
- net N$7: track 0.00 -> 11.5 mm
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
Commit message: Circuito
Aumentado el grosor de algunas pistas.
Parts:
- moved Q4 5.00 mm to (15.4, 42.6)
- moved R3 4.27 mm to (14.0, 60.0)
- moved R7 4.27 mm to (14.0, 56.0)
- moved R4 3.81 mm to (26.0, 59.0)
- moved R8 3.81 mm to (26.0, 55.0)
- moved Q3 3.50 mm to (28.7, 42.1)
Routing:
- net N$13: track 39.1 -> 45.4 mm
- net N$16: track 100.9 -> 94.7 mm
- net GND: track 247.5 -> 243.6 mm
- net N$8: track 36.8 -> 33.5 mm
- net N$9: track 12.7 -> 9.44 mm
- net N$11: track 155.0 -> 152.3 mm
- net N$12: track 102.4 -> 104.7 mm
- net N$15: track 60.6 -> 62.3 mm
- net N$14: track 51.5 -> 52.8 mm
- net N$17: track 66.8 -> 65.8 mm
- net N$10: track 13.8 -> 12.9 mm
Other:
- board text added: "+Vb"
- board text removed: "+11.1V"
